Commit message: enable test and retrain modes for laikago, mirror ANYmal file structure

File: raisim_gym/env/env/laikago/laikago/urdf/laikago.urdf (robot description, URDF)
Before this commit: robot laikago_description, 21 links, 20 joints
Links:
- link FL_calf: geometry collision box size=0.25 0.016 0.016; visual mesh filename=../meshes/calf.dae scale=1 1 1
- link FL_hip: geometry collision cylinder length=0.08 radius=0.041; visual mesh filename=../meshes/hip.dae scale=1 1 1
- link FL_thigh: geometry collision box size=0.25 0.034 0.043; visual mesh filename=../meshes/thigh.dae scale=1 1 1
- link FR_calf: geometry collision box size=0.25 0.016 0.016; visual mesh filename=../meshes/calf.dae scale=1 1 1
- link FR_hip: geometry collision cylinder length=0.08 radius=0.041; visual mesh filename=../meshes/hip.dae scale=1 1 1
- link FR_thigh: geometry collision box size=0.25 0.034 0.043; visual mesh filename=../meshes/thigh_mirror.dae scale=1 1 1
- link RL_calf: geometry collision box size=0.25 0.016 0.016; visual mesh filename=../meshes/calf.dae scale=1 1 1
- link RL_hip: geometry collision cylinder length=0.08 radius=0.041; visual mesh filename=../meshes/hip.dae scale=1 1 1
- link RL_thigh: geometry collision box size=0.25 0.034 0.043; visual mesh filename=../meshes/thigh.dae scale=1 1 1
- link RR_calf: geometry collision box size=0.25 0.016 0.016; visual mesh filename=../meshes/calf.dae scale=1 1 1
- link RR_hip: geometry collision cylinder length=0.08 radius=0.041; visual mesh filename=../meshes/hip.dae scale=1 1 1
- link RR_thigh: geometry collision box size=0.25 0.034 0.043; visual mesh filename=../meshes/thigh_mirror.dae scale=1 1 1
- link trunk: geometry collision box size=0.5616 0.172 0.1875; visual mesh filename=../meshes/trunk.dae scale=1 1 1
